Commit message: Comment out prop2 definitions in Single-Agent-Def.xacro
Ducted fan UAV uses single propeller per module.
prop2_link and actuator_prop2_joint are commented out
but preserved for reference.

File: src/tvmd/urdf/Single-Agent-Def.xacro (robot description, xacro)
@@ -90,4 +90,5 @@
   <xacro:gz_material joint_name="module${module_id}_prop1_link" color_name="Yellow" />
 </xacro:macro>
+<!-- prop2_link removed for ducted fan UAV (single propeller per module)
 <xacro:macro name="prop2_link" params="module_id">
   <link name="module${module_id}_prop2_link">
@@ -113,4 +114,5 @@
   <xacro:gz_material joint_name="module${module_id}_prop2_link" color_name="Yellow" />
 </xacro:macro>
+-->
 <!-- Joints -->
 <!-- Y-Servo -->
@@ -165,4 +167,5 @@
     number_motor="${module_id*2-2}"/>
 </xacro:macro>
+<!-- actuator_prop2_joint removed for ducted fan UAV (single propeller per module)
 <xacro:macro name="actuator_prop2_joint" params="module_id">
   <joint name="module${module_id}_actuator_prop2_joint" type="continuous">
@@ -172,5 +175,4 @@
     <axis xyz="0.0 0.0 -1.0"/>
     <limit effort="30000" velocity="10000.0" lower="-1e+16" upper="1e+16" />
-    <!-- <limit lower="-1e+16" upper="1e+16" /> -->
   </joint>
   <xacro:simple_transmission joint_name="module${module_id}_actuator_prop2_joint" />
@@ -179,3 +181,4 @@
     number_motor="${module_id*2-1}"/>
 </xacro:macro>
+-->
 </robot>

Commit message: Refactor to single propeller per agent
- Remove prop2_link and actuator_prop2_joint from Single-Agent-Def.xacro
- Update motor numbering from module_id*2-2 to module_id-1
- Remove prop2 macro calls from tvmd.xacro module definition
- Update republisher.py joint indexing for 3 joints per module
- Reduce motor count from 8 to 4 (one per agent)

https://claude.ai/code/session_01Jw14ek9ymbLHkeU4kCpkH7

File: src/tvmd/urdf/Single-Agent-Def.xacro (robot description, xacro)
@@ -90,27 +90,4 @@
   <xacro:gz_material joint_name="module${module_id}_prop1_link" color_name="Yellow" />
 </xacro:macro>
-<xacro:macro name="prop2_link" params="module_id">
-  <link name="module${module_id}_prop2_link">
-    <inertial>
-      <origin xyz="0.0 0.0 0.0" rpy="0 0 0"/>
-      <mass value="0.00253778"/>
-      <inertia ixx="0.00000702" iyy="0.00000005" izz="0.00000705" ixy="0.00000000" iyz="-0.00000009" ixz="0.00000000"/>
-    </inertial>
-    <visual>
-      <origin xyz="0.0 0.0 0.0" rpy="${pi/2} 0 0"/>
-      <geometry>
-        <mesh filename="package://tvmd/meshes/agent/Propeller_9047.stl" scale="0.001 0.001 0.001"/>
-      </geometry>
-      <material name="yellow"/>
-    </visual>
-    <collision name='module${module_id}_rotor_2_collision'>
-      <origin xyz="0 0 0" rpy="0 0 0"/>
-      <geometry>
-        <cylinder length="0.005" radius="0.12"/>
-      </geometry>
-    </collision>
-  </link>
-  <xacro:gz_material joint_name="module${module_id}_prop2_link" color_name="Yellow" />
-</xacro:macro>
 <!-- Joints -->
 <!-- Y-Servo -->
@@ -163,19 +140,5 @@
   <xacro:gz_prop joint_name="module${module_id}_actuator_prop1_joint"
     link_name="module${module_id}_prop1_link"
-    number_motor="${module_id*2-2}"/>
-</xacro:macro>
-<xacro:macro name="actuator_prop2_joint" params="module_id">
-  <joint name="module${module_id}_actuator_prop2_joint" type="continuous">
-    <origin xyz="0.0 0.0 -0.0781" rpy="0 0 0"/>
-    <parent link="module${module_id}_actuator_link"/>
-    <child link="module${module_id}_prop2_link"/>
-    <axis xyz="0.0 0.0 -1.0"/>
-    <limit effort="30000" velocity="10000.0" lower="-1e+16" upper="1e+16" />
-    <!-- <limit lower="-1e+16" upper="1e+16" /> -->
-  </joint>
-  <xacro:simple_transmission joint_name="module${module_id}_actuator_prop2_joint" />
-  <xacro:gz_prop joint_name="module${module_id}_actuator_prop2_joint"
-    link_name="module${module_id}_prop2_link"
-    number_motor="${module_id*2-1}"/>
+    number_motor="${module_id-1}"/>
 </xacro:macro>
 </robot>

File: src/tvmd/urdf/tvmd.xacro (robot description, xacro)
@@ -13,10 +13,8 @@
   <xacro:actuator_link module_id="${module_id}" />
   <xacro:prop1_link module_id="${module_id}" />
-  <xacro:prop2_link module_id="${module_id}" />
   <!-- Joints -->
   <xacro:body_gimbal_joint module_id="${module_id}" />
   <xacro:gimbal_actuator_joint module_id="${module_id}" />
   <xacro:actuator_prop1_joint module_id="${module_id}" />
-  <xacro:actuator_prop2_joint module_id="${module_id}" />
 </xacro:macro>
 <!-- Team System -->
