Commit message: Convert TVMD to TVHQ configuration and update px4_msgs

File: src/tvmd/urdf/Navigator-Def.xacro (robot description, xacro)
@@ -13,5 +13,5 @@
             <mesh filename="package://tvmd/meshes/navigator/NavigatorModule-Sim.stl" scale="0.001 0.001 0.001"/>
             </geometry>
-            <material name="dark_blue"/>
+            <material name="titanium_purple"/>
         </visual>
         <collision>

File: src/tvmd/urdf/materials.xacro (robot description, xacro)
@@ -1,18 +1,54 @@
 <?xml version="1.0" ?>
 <robot name="tvmd" xmlns:xacro="http://www.ros.org/wiki/xacro" >
-<material name="silver">
-  <color rgba="0.700 0.700 0.700 1.000"/>
-</material>
-<material name="yellow">
-  <color rgba="1.000 1.000 0.000 1.000"/>
-</material>
-<material name="black">
-  <color rgba="0.000 0.000 0.000 1.000"/>
-</material>
-<material name="gray">
-  <color rgba="0.200 0.200 0.200 1.000"/>
-</material>
-<material name="dark_blue">
-  <color rgba="0.100 0.100 0.300 1.000"/>
-</material>
+  <material name="silver">
+    <color rgba="0.700 0.700 0.700 1.000"/>
+  </material>
+  <material name="aluminum">
+    <color rgba="0.800 0.800 0.820 1.000"/>
+  </material>
+  <material name="dark_metal">
+    <color rgba="0.300 0.300 0.320 1.000"/>
+  </material>
+  <material name="gold">
+    <color rgba="0.830 0.680 0.210 1.000"/>
+  </material>
+  <material name="copper">
+    <color rgba="0.720 0.450 0.200 1.000"/>
+  </material>
+  <material name="carbon_fiber">
+    <color rgba="0.150 0.150 0.150 1.000"/>
+  </material>
+  <material name="titanium_blue">
+    <color rgba="0.300 0.350 0.500 1.000"/>
+  </material>
+  <material name="titanium_purple">
+    <color rgba="0.450 0.350 0.500 1.000"/>
+  </material>
+  <material name="titanium_rainbow">
+    <color rgba="0.500 0.400 0.450 1.000"/>
+  </material>
+  <material name="red">
+    <color rgba="0.800 0.200 0.200 1.000"/>
+  </material>
+  <material name="orange">
+    <color rgba="1.000 0.500 0.000 1.000"/>
+  </material>
+  <material name="yellow">
+    <color rgba="1.000 1.000 0.000 1.000"/>
+  </material>
+  <material name="green">
+    <color rgba="0.200 0.800 0.200 1.000"/>
+  </material>
+  <material name="blue">
+    <color rgba="0.200 0.200 0.800 1.000"/>
+  </material>
+  <material name="black">
+    <color rgba="0.000 0.000 0.000 1.000"/>
+  </material>
+  <material name="gray">
+    <color rgba="0.200 0.200 0.200 1.000"/>
+  </material>
+  <material name="dark_blue">
+    <color rgba="0.100 0.100 0.300 1.000"/>
+  </material>
 </robot>

File: src/tvmd/urdf/model.urdf (robot description, URDF)
Before this commit: robot tvmd, 22 links, 21 joints
Links:
- removed link module1_prop2_link
- removed link module2_prop2_link
- removed link module3_prop2_link
- removed link module4_prop2_link
- link module1_body_link: mass 0.50823179 -> 0.1; geometry 
- link module2_body_link: mass 0.50823179 -> 0.1; geometry 
- link module3_body_link: mass 0.50823179 -> 0.1; geometry 
- link module4_body_link: mass 0.50823179 -> 0.1; geometry 
Joints:
- removed joint module1_actuator_prop2_joint
- removed joint module2_actuator_prop2_joint
- removed joint module3_actuator_prop2_joint
- removed joint module4_actuator_prop2_joint
- joint module1_actuator_prop1_joint: origin xyz=0.0 0.0 0.0781 rpy=0 0 0 -> xyz=0.0 0.0 0.0 rpy=0 0 0
- joint module1_body_gimbal_joint: limit lower=-1.5707963267948966 upper=1.5707963267948966 effort=30000 velocity=10.0 -> lower=-0.7853981633974483 upper=0.7853981633974483 effort=30000 velocity=10.0; origin xyz=0.0 0.0 0.068 rpy=0 0 0 -> xyz=0.0 0.0 0.0 rpy=0 0 0
- joint module1_gimbal_actuator_joint: limit lower=-0.5235987755982988 upper=0.5235987755982988 effort=30000 velocity=10.0 -> lower=-0.349 upper=0.349 effort=30000 velocity=10.0
- joint module2_actuator_prop1_joint: origin xyz=0.0 0.0 0.0781 rpy=0 0 0 -> xyz=0.0 0.0 0.0 rpy=0 0 0
- joint module2_body_gimbal_joint: limit lower=-1.5707963267948966 upper=1.5707963267948966 effort=30000 velocity=10.0 -> lower=-0.7853981633974483 upper=0.7853981633974483 effort=30000 velocity=10.0; origin xyz=0.0 0.0 0.068 rpy=0 0 0 -> xyz=0.0 0.0 0.0 rpy=0 0 0
- joint module2_gimbal_actuator_joint: limit lower=-0.5235987755982988 upper=0.5235987755982988 effort=30000 velocity=10.0 -> lower=-0.349 upper=0.349 effort=30000 velocity=10.0
- joint module3_actuator_prop1_joint: origin xyz=0.0 0.0 0.0781 rpy=0 0 0 -> xyz=0.0 0.0 0.0 rpy=0 0 0
- joint module3_body_gimbal_joint: limit lower=-1.5707963267948966 upper=1.5707963267948966 effort=30000 velocity=10.0 -> lower=-0.7853981633974483 upper=0.7853981633974483 effort=30000 velocity=10.0; origin xyz=0.0 0.0 0.068 rpy=0 0 0 -> xyz=0.0 0.0 0.0 rpy=0 0 0
- joint module3_gimbal_actuator_joint: limit lower=-0.5235987755982988 upper=0.5235987755982988 effort=30000 velocity=10.0 -> lower=-0.349 upper=0.349 effort=30000 velocity=10.0
- joint module4_actuator_prop1_joint: origin xyz=0.0 0.0 0.0781 rpy=0 0 0 -> xyz=0.0 0.0 0.0 rpy=0 0 0
- joint module4_body_gimbal_joint: limit lower=-1.5707963267948966 upper=1.5707963267948966 effort=30000 velocity=10.0 -> lower=-0.7853981633974483 upper=0.7853981633974483 effort=30000 velocity=10.0; origin xyz=0.0 0.0 0.068 rpy=0 0 0 -> xyz=0.0 0.0 0.0 rpy=0 0 0
- joint module4_gimbal_actuator_joint: limit lower=-0.5235987755982988 upper=0.5235987755982988 effort=30000 velocity=10.0 -> lower=-0.349 upper=0.349 effort=30000 velocity=10.0
- joint rigid_base_link_module1_body_link: origin xyz=0.215 0.215 0.0 rpy=0 0 1.5707963267948966 -> xyz=0.1675 0.1825 -0.02 rpy=0 0 0
- joint rigid_base_link_module2_body_link: origin xyz=0.215 -0.215 0.0 rpy=0 0 1.5707963267948966 -> xyz=0.1675 -0.172 -0.02 rpy=0 0 0
- joint rigid_base_link_module3_body_link: origin xyz=-0.215 0.215 0.0 rpy=0 0 0 -> xyz=-0.15 0.1825 -0.02 rpy=0 0 0
- joint rigid_base_link_module4_body_link: origin xyz=-0.215 -0.215 0.0 rpy=0 0 0 -> xyz=-0.15 -0.175 -0.02 rpy=0 0 0

File: src/tvmd/urdf/orig/Single-Agent-Def.xacro (robot description, xacro)
@@ -7,14 +7,14 @@
     <inertial>
       <origin xyz="0.0 0.0 0.0" rpy="0 0 0"/>
-      <mass value="0.1"/>
+      <mass value="0.50823179"/>
       <inertia ixx="0.01671968" iyy="0.00290137" izz="0.01758533" ixy="-0.00001217" iyz="-0.00003388" ixz="-0.00000326"/>
     </inertial>
-    <!-- <visual>
-      <origin xyz="0 0 0" rpy="-1.5708 0 0"/>
+    <visual>
+      <origin xyz="0 0 0" rpy="0 0 0"/>
       <geometry>
         <mesh filename="package://tvmd/meshes/agent/base_link.stl" scale="0.001 0.001 0.001"/>
       </geometry>
       <material name="black"/>
-    </visual> -->
+    </visual>
     <!-- <collision>
       <origin xyz="0 0 0" rpy="0 0 0"/>
@@ -35,12 +35,12 @@
     </inertial>
     <visual>
-      <origin xyz="-0.001 -0.02 0.065" rpy=" 0 0 0"/>
+      <origin xyz="0.0 0.0 -0.068" rpy="0 0 0"/>
       <geometry>
         <mesh filename="package://tvmd/meshes/agent/Gimbal_Frame_1.stl" scale="0.001 0.001 0.001"/>
       </geometry>
-      <material name="copper"/>
+      <material name="gray"/>
     </visual>
     <collision name='module${module_id}_actuator_collision'>
-      <origin xyz="0.001 -0.018 0.065" rpy="0 0 0"/>
+      <origin xyz="0 0 0" rpy="${pi/2} 0 0"/>
       <geometry>
         <cylinder length="0.400" radius="0.010"/>
@@ -58,10 +58,9 @@
     </inertial>
     <visual>
-      <!-- <origin xyz="0.0 0.17 0.0" rpy="1.5708 0 0"/> -->
-      <origin xyz="0.0 0.185 0.0" rpy="1.5708 0 0"/>
+      <origin xyz="0.0 0.0 -0.068" rpy="0 0 0"/>
       <geometry>
         <mesh filename="package://tvmd/meshes/agent/Actuator_1.stl" scale="0.001 0.001 0.001"/>
       </geometry>
-      <material name="red"/>
+      <material name="gray"/>
     </visual>
   </link>
@@ -76,9 +75,9 @@
     </inertial>
     <visual>
-      <origin xyz="0.0 0 0.035" rpy="1.5708 0 0"/>
+      <origin xyz="0.0 0.0 0.0" rpy="${pi/2} 0 0"/>
       <geometry>
         <mesh filename="package://tvmd/meshes/agent/Propeller_9047.stl" scale="0.001 0.001 0.001"/>
       </geometry>
-      <material name="gold"/>
+      <material name="yellow"/>
     </visual>
     <collision name='module${module_id}_rotor_1_collision'>
@@ -91,5 +90,5 @@
   <xacro:gz_material joint_name="module${module_id}_prop1_link" color_name="Yellow" />
 </xacro:macro>
-<!-- <xacro:macro name="prop2_link" params="module_id">
+<xacro:macro name="prop2_link" params="module_id">
   <link name="module${module_id}_prop2_link">
     <inertial>
@@ -113,10 +112,10 @@
   </link>
   <xacro:gz_material joint_name="module${module_id}_prop2_link" color_name="Yellow" />
-</xacro:macro> -->
+</xacro:macro>
 <!-- Joints -->
 <!-- Y-Servo -->
 <xacro:macro name="body_gimbal_joint" params="module_id">
   <joint name="module${module_id}_body_gimbal_joint" type="revolute">
-    <origin xyz="0.0 0.0 0.0" rpy="0 0 0"/>
+    <origin xyz="0.0 0.0 0.068" rpy="0 0 0"/>
     <parent link="module${module_id}_body_link"/>
     <child link="module${module_id}_gimbal_link"/>
@@ -154,5 +153,5 @@
 <xacro:macro name="actuator_prop1_joint" params="module_id">
   <joint name="module${module_id}_actuator_prop1_joint" type="continuous">
-    <origin xyz="0.0 0.0 0.0" rpy="0 0 0"/>
+    <origin xyz="0.0 0.0 0.0781" rpy="0 0 0"/>
     <parent link="module${module_id}_actuator_link"/>
     <child link="module${module_id}_prop1_link"/>
@@ -164,19 +163,19 @@
   <xacro:gz_prop joint_name="module${module_id}_actuator_prop1_joint"
     link_name="module${module_id}_prop1_link"
-    number_motor="${module_id-1}"/>
+    number_motor="${module_id*2-2}"/>
 </xacro:macro>
-<!-- <xacro:macro name="actuator_prop2_joint" params="module_id"> -->
-  <!-- <joint name="module${module_id}_actuator_prop2_joint" type="continuous"> -->
-    <!-- <origin xyz="0.0 0.0 -0.0781" rpy="0 0 0"/> -->
-    <!-- <parent link="module${module_id}_actuator_link"/>
+<xacro:macro name="actuator_prop2_joint" params="module_id">
+  <joint name="module${module_id}_actuator_prop2_joint" type="continuous">
+    <origin xyz="0.0 0.0 -0.0781" rpy="0 0 0"/>
+    <parent link="module${module_id}_actuator_link"/>
     <child link="module${module_id}_prop2_link"/>
     <axis xyz="0.0 0.0 -1.0"/>
-    <limit effort="30000" velocity="10000.0" lower="-1e+16" upper="1e+16" /> -->
+    <limit effort="30000" velocity="10000.0" lower="-1e+16" upper="1e+16" />
     <!-- <limit lower="-1e+16" upper="1e+16" /> -->
-  <!-- </joint> -->
-  <!-- <xacro:simple_transmission joint_name="module${module_id}_actuator_prop2_joint" />
+  </joint>
+  <xacro:simple_transmission joint_name="module${module_id}_actuator_prop2_joint" />
   <xacro:gz_prop joint_name="module${module_id}_actuator_prop2_joint"
     link_name="module${module_id}_prop2_link"
-    number_motor="${module_id*2-1}"/> -->
-<!-- </xacro:macro> -->
+    number_motor="${module_id*2-1}"/>
+</xacro:macro>
 </robot>

File: src/tvmd/urdf/orig/tvmd.xacro (robot description, xacro)
@@ -13,10 +13,10 @@
   <xacro:actuator_link module_id="${module_id}" />
   <xacro:prop1_link module_id="${module_id}" />
-  <!-- <xacro:prop2_link module_id="${module_id}" /> -->
+  <xacro:prop2_link module_id="${module_id}" />
   <!-- Joints -->
   <xacro:body_gimbal_joint module_id="${module_id}" />
   <xacro:gimbal_actuator_joint module_id="${module_id}" />
   <xacro:actuator_prop1_joint module_id="${module_id}" />
-  <!-- <xacro:actuator_prop2_joint module_id="${module_id}" /> -->
+  <xacro:actuator_prop2_joint module_id="${module_id}" />
 </xacro:macro>
 <!-- Team System -->
@@ -26,5 +26,5 @@
 <xacro:module module_id="3" />
 <xacro:module module_id="4" />
-<!-- <xacro:rigid_connection
+<xacro:rigid_connection
   parent="base_link" child="module1_body_link"
   pos_x="0.215" pos_y="0.215" pos_z="0.0" z_psi="${pi/2}" />
@@ -37,21 +37,4 @@
 <xacro:rigid_connection
   parent="base_link" child="module4_body_link"
-  pos_x="-0.215" pos_y="-0.215" pos_z="0.0" z_psi="0" /> -->
-<!-- Module positions matching PX4 CA_MDx parameters -->
-<!-- MD0: Front-Left -->
-<xacro:rigid_connection
-  parent="base_link" child="module1_body_link"
-  pos_x="0.1675" pos_y="0.1825" pos_z="-0.02" z_psi="0" />
-<!-- MD1: Front-Right -->
-<xacro:rigid_connection
-  parent="base_link" child="module2_body_link"
-  pos_x="0.1675" pos_y="-0.172" pos_z="-0.02" z_psi="0" />
-<!-- MD2: Rear-Left -->
-<xacro:rigid_connection
-  parent="base_link" child="module3_body_link"
-  pos_x="-0.15" pos_y="0.1825" pos_z="-0.02" z_psi="0" />
-<!-- MD3: Rear-Right -->
-<xacro:rigid_connection
-  parent="base_link" child="module4_body_link"
-  pos_x="-0.15" pos_y="-0.175" pos_z="-0.02" z_psi="0" />
+  pos_x="-0.215" pos_y="-0.215" pos_z="0.0" z_psi="0" />
 </robot>
